Commit message: add actual fred.urdf compiled from the xacro file, oops.

File: urdf/fred.urdf (robot description, URDF)
Before this commit: robot kuka_lwr, 4 links, 3 joints
Links:
- added link gripper; visual mesh filename=file:///home/thomas/tutorial_ws/urdf_tutorial/urdf/meshes_f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 scale=0.001 0.001 0.001
- added link wrist; visual mesh filename=file:///home/thomas/tutorial_ws/urdf_tutorial/urdf/meshes_f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 scale=0.001 0.001 0.001
- added link wrist_servo; visual mesh filename=file:///home/thomas/tutorial_ws/urdf_tutorial/urdf/meshes_f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 scale=0.001 0.001 0.001
Joints:
- added joint arm_upper_to_wrist: type continuous, parent arm_upper, child wrist, origin xyz=0 0.102 0, axis 0 1 0
- added joint wrist_servo_to_gripper: type continuous, parent wrist_servo, child gripper, origin xyz=0 0.017 0, axis 0 1 0
- added joint wrist_to_wrist_servo: type continuous, parent wrist, child wrist_servo, origin xyz=0 0.11625 0, axis 1 0 0
