Commit message: wip position recorder

File: src/simulation/urdf/fred_with_spheres_new.urdf (robot description, URDF)
Before this commit: robot fred, 10 links, 9 joints
Joints:
- joint base_plate_to_arm_lower: limit lower=0.0 upper=3.14159265359 effort=1000.0 velocity=10 -> lower=-3.14159265359 upper=3.14159265359 effort=1000.0 velocity=10
